File: garagesp.kicad_sch (KiCad schematic)
At the start: 20 parts, among them J1 USB_C_Receptacle_USB2.0_14P, J2 AHT21, J3 DOOR CTL, J4 DOOR SW, K1 SANYOU_SRD_Form_C, Q1 BC547, SW1 RESET, SW2 BOOT, U1 ESP32-C3-WROOM-02, U2 AP2112K-3.3

Commit message: move things around again
Parts:
- added D1: B120-E3, Diode_SMD:D_SMA, symbol Diode:B120-E3
Connections:
- net GND: now also D1.2 (A)
- net at K1.2, Q1.3 (E): now also D1.1 (K)
- net 3.3 renamed 3V3
- net 5 renamed 5V
Other:
- moved on the sheet: C1, C2, C3, J1, J2, J3, J4, K1, Q1, R1, R2, R3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

Commit message: finalize placements, add LCSC part #s
Parts:
- removed K1: SANYOU_SRD_Form_C, Relay_THT:Relay_SPDT_SANYOU_SRD_Series_Form_C, symbol Relay:SANYOU_SRD_Form_C
- added K1: SANYOU_SRD_Form_A, Relay_THT:Relay_SPST_SANYOU_SRD_Series_Form_A, symbol Relay:SANYOU_SRD_Form_A
- C1, C3: LCSC (none) -> C1713
- C2: value 0.1uF -> 100 nF; LCSC (none) -> C476766
- D1: LCSC (none) -> C2902910
- J1: LCSC (none) -> C2894897
- J2: LCSC (none) -> C52016392
- J3, J4: LCSC (none) -> C192562
- Q1: LCSC (none) -> C47089404
- R1, R2: LCSC (none) -> C27834
- R3, R4, R5: LCSC (none) -> C17414
- R6: renamed from R7; LCSC (none) -> C17414
- R7: renamed from R6; LCSC (none) -> C17517
- SW1, SW2: footprint Button_Switch_SMD:SW_SPST_CK_RS282G05A3 -> Button_Switch_SMD:SW_SPST_TS-1088-xR020; LCSC (none) -> C720477
- U1: LCSC (none) -> C2934560
- U2: LCSC (none) -> C23380830
Connections:
- net CTL1: now also K1.1
- net CTL2: now also K1.3
- net GND: now also K1.5
- net at D1.1 (K), Q1.3 (E): now also K1.2
Other:
- moved on the sheet: D1

Commit message: finalize more things
Parts:
- C1: renamed from C3; LCSC C1713 -> C15850
- C2: renamed from C1; LCSC C1713 -> C15850
- C3: renamed from C2; LCSC C476766 -> C28233
- R7: value 2.1k -> 5.1k; LCSC C17517 -> C27834
Changed lines of the file:
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@@
+	)
+	(symbol
+		(lib_id "Device:R")
+		(at 189.23 133.35 90)
+		(unit 1)
+		(exclude_from_sim no)
+		(in_bom yes)
+		(on_board yes)
+		(dnp no)
+		(fields_autoplaced yes)
+		(property "Reference" "R7"
+			(at 189.23 127 90)
+			(effects
+				(font
+					(size 1.27 1.27)
+				)
+			)
+		)
+		(property "Value" "5.1k"
+			(at 189.23 129.54 90)
+			(effects
+				(font
+					(size 1.27 1.27)
+				)
+			)
+		)
+		(property "Footprint" "Resistor_SMD:R_0805_2012Metric_Pad1.20x1.40mm_HandSolder"
+			(at 189.23 135.128 90)
+			(effects
+				(font
+					(size 1.27 1.27)
+				)
+				(hide yes)
+			)
+		)
+		(property "Datasheet" "~"
+			(at 189.23 133.35 0)
+			(effects
+				(font
+					(size 1.27 1.27)
+				)
+				(hide yes)
+			)
+		)
+		(property "Description" "Resistor"
+			(at 189.23 133.35 0)
+			(effects
+				(font
+					(size 1.27 1.27)
+				)
+				(hide yes)
+			)
+		)
+		(property "LCSC" "C27834"
+			(at 189.23 133.35 90)
+			(effects
+				(font
+					(size 1.27 1.27)
+				)
+				(hide yes)
+			)
+		)
+		(pin "2"
+		)
+		(pin "1"
+		)
+		(instances
+			(project "garagesp"
+				(path "/3fa1ee2a-4fd2-4656-a08a-79cff3e38c75"
+					(reference "R7")
+					(unit 1)
+				)
+			)
+		)
 	)
 	(symbol
@@
 		(dnp no)
 		(fields_autoplaced yes)
-		(property "Reference" "C2"
+		(property "Reference" "C3"
 			(at 148.59 147.3199 0)
 			(effects
@@
 			)
 		)
-		(property "LCSC" "C476766"
+		(property "LCSC" "C28233"
 			(at 144.78 148.59 0)
 			(effects
@@
 			(project "garagesp"
 				(path "/3fa1ee2a-4fd2-4656-a08a-79cff3e38c75"
-					(reference "C2")
+					(reference "C3")
 					(unit 1)
 				)
@@
 		(dnp no)
 		(fields_autoplaced yes)
-		(property "Reference" "C3"
+		(property "Reference" "C1"
 			(at 107.95 147.3199 0)
 			(effects
@@
 			)
 		)
-		(property "LCSC" "C1713"
+		(property "LCSC" "C15850"
 			(at 104.14 148.59 0)
 			(effects
@@
 			(project "garagesp"
 				(path "/3fa1ee2a-4fd2-4656-a08a-79cff3e38c75"
-					(reference "C3")
+					(reference "C1")
 					(unit 1)
 				)
@@
 	)
 	(symbol
-		(lib_id "Device:R")
-		(at 189.23 133.35 90)
-		(unit 1)
-		(exclude_from_sim no)
-		(in_bom yes)
-		(on_board yes)
-		(dnp no)
-		(fields_autoplaced yes)
-		(property "Reference" "R7"
-			(at 189.23 127 90)
-			(effects
-				(font
-					(size 1.27 1.27)
-				)
-			)
-		)
-		(property "Value" "2.1k"
-			(at 189.23 129.54 90)
-			(effects
-				(font
-					(size 1.27 1.27)
-				)
-			)
-		)
-		(property "Footprint" "Resistor_SMD:R_0805_2012Metric_Pad1.20x1.40mm_HandSolder"
-			(at 189.23 135.128 90)
-			(effects
-				(font
-					(size 1.27 1.27)
-				)
-				(hide yes)
-			)
-		)
-		(property "Datasheet" "~"
-			(at 189.23 133.35 0)
-			(effects
-				(font
-					(size 1.27 1.27)
-				)
-				(hide yes)
-			)
-		)
-		(property "Description" "Resistor"
-			(at 189.23 133.35 0)
-			(effects
-				(font
-					(size 1.27 1.27)
-				)
-				(hide yes)
-			)
-		)
-		(property "LCSC" " C17517 "
-			(at 189.23 133.35 90)
-			(effects
-				(font
-					(size 1.27 1.27)
-				)
-				(hide yes)
-			)
-		)
-		(pin "1"
-		)
-		(pin "2"
-		)
-		(instances
-			(project "garagesp"
-				(path "/3fa1ee2a-4fd2-4656-a08a-79cff3e38c75"
-					(reference "R7")
-					(unit 1)
-				)
-			)
-		)
-	)
-	(symbol
 		(lib_id "Transistor_BJT:BC547")
 		(at 200.66 133.35 0)
@@
 		(dnp no)
 		(fields_autoplaced yes)
-		(property "Reference" "C1"
+		(property "Reference" "C2"
 			(at 137.16 147.3199 0)
 			(effects
@@
 			)
 		)
-		(property "LCSC" "C1713"
+		(property "LCSC" "C15850"
 			(at 133.35 148.59 0)
 			(effects
@@
 			(project ""
 				(path "/3fa1ee2a-4fd2-4656-a08a-79cff3e38c75"
-					(reference "C1")
-					(unit 1)
-				)
+					(reference "C2")
+					(unit 1)
+				)

Commit message: update schematics
Parts:
- added C4, C5: 100 nF, Capacitor_SMD:C_0805_2012Metric_Pad1.18x1.45mm_HandSolder, symbol Device:C
- added FB1: FerriteBead, symbol Device:FerriteBead
- added R10: 10k, Resistor_SMD:R_0805_2012Metric_Pad1.20x1.40mm_HandSolder, symbol Device:R
- added R11, R12: 220, Resistor_SMD:R_0805_2012Metric_Pad1.20x1.40mm_HandSolder, symbol Device:R
- added R8, R9: 2.1k, Resistor_SMD:R_0805_2012Metric_Pad1.20x1.40mm_HandSolder, symbol Device:R
- C3: value 100 nF -> 10uF; LCSC C28233 -> C15850
Connections:
- net 3V3: no longer C2.1, C3.1, J2.1 (Pin_1), U1.1 (3V3), U2.5 (VOUT)
- net GND: now also C4.2, C5.2, FB1.2, R10.1, R11.2, R12.2; no longer J1.S1 (SHIELD), SW1.2, SW2.2
- net RELAY: now also R10.2
- net SCL: now also R8.1
- net SDA: now also R9.1
- net 5V renamed +5V
- net +5V: now also FB1.1
- new net: R12.1, SW1.2
- new net: R11.1, SW2.2
- new net +3V3: C2.1, C3.1, C4.1, C5.1, J2.1 (Pin_1), R8.2, R9.2, U1.1 (3V3), U2.5 (VOUT)
- no-connect marks 0 -> 7
Other:
- moved on the sheet: J1, J2, J3, R1, R2, R3, R4, R5, R6, SW1, SW2, U1

Commit message: add capacitors and resistors
Parts:
- removed C3: 10uF, Capacitor_SMD:C_0805_2012Metric_Pad1.18x1.45mm_HandSolder, symbol Device:C
- removed Q1: BC547, Package_TO_SOT_THT:TO-92_Inline, symbol Transistor_BJT:BC547
- removed U2: AP2112K-3.3, Package_TO_SOT_SMD:SOT-23-5, symbol Regulator_Linear:AP2112K-3.3
- added C10, C7: 100nF, Capacitor_SMD:C_0805_2012Metric_Pad1.18x1.45mm_HandSolder, symbol Device:C
- added C11: 4.7uF, symbol Device:C_Polarized
- added C4, C6: 10uF, Capacitor_SMD:C_0805_2012Metric_Pad1.18x1.45mm_HandSolder, symbol Device:C
- added C9: 10nF, Capacitor_SMD:C_0603_1608Metric_Pad1.08x0.95mm_HandSolder, symbol Device:C
- added D2: RED LED, LED_SMD:LED_0603_1608Metric_Pad1.05x0.95mm_HandSolder, symbol Device:LED
- added D3, D4, D5: GREEN LED, LED_SMD:LED_0603_1608Metric_Pad1.05x0.95mm_HandSolder, symbol Device:LED
- added Q1, Q2: SS8050, Package_TO_SOT_SMD:SOT-23, symbol Transistor_BJT:SS8050
- added R13: 10k, Resistor_SMD:R_0805_2012Metric_Pad1.20x1.40mm_HandSolder, symbol Device:R
- added R14: 220, Resistor_SMD:R_0805_2012Metric_Pad1.20x1.40mm_HandSolder, symbol Device:R
- added U2: AMS1117-3.3, Package_TO_SOT_SMD:SOT-223-3_TabPin2, symbol Regulator_Linear:AMS1117-3.3
- added U3: USBLC6-2SC6, Package_TO_SOT_SMD:SOT-23-6, symbol Power_Protection:USBLC6-2SC6
- added U4: PC817, Package_DIP:DIP-4_W7.62mm, symbol Isolator:PC817
- C3: renamed from C4; value 100 nF -> 100nF
- C5: value 100 nF -> 100nF
- FB1: value FerriteBead -> 70mΩ 33Ω@100MHz; footprint (none) -> Inductor_SMD:L_0805_2012Metric_Pad1.05x1.20mm_HandSolder; symbol Device:FerriteBead -> Device:FerriteBead_Small; LCSC (none) -> C74764
- R10: value 10k -> 1k; LCSC C17414 -> (none)
- R7: value 5.1k -> 100; LCSC C27834 -> (none)
- SW1: value RESET -> ~
- SW2: value BOOT -> ~
Connections:
- net +3V3: now also D1.1 (K), K1.5, R11.1, R12.2, R3.2, R4.1, R5.2, R6.1, C4.1, R13.2, U2.2 (VO), U4.4
- net +5V: now also C10.1, C11.1, R14.2, U2.3 (VI); no longer J1.A4 (VBUS), J1.A9 (VBUS), J1.B4 (VBUS), J1.B9 (VBUS)
- net GND: now also SW1.1, SW2.1, C10.2, C11.2, C4.2, C6.2, C7.1, C9.2, D2.1 (K), D3.1 (K), D4.1 (K), Q1.2 (E), Q2.2 (E), U2.1 (GND), U3.2 (GND); no longer D1.2 (A), FB1.2, K1.5, R10.1, R11.2, R12.2
- net RELAY: now also R7.2; no longer R10.2, R7.1
- net SCL: now also R9.1, U1.3 (IO4); no longer R8.1, U1.4 (IO5)
- net SDA: now also R8.1, U1.4 (IO5); no longer R9.1, U1.3 (IO4)
- net SW: now also D5.1 (K), Q2.3 (C); no longer J4.1 (Pin_1)
- net at R12.1: now also D3.2 (A); no longer SW1.2
- net at R2.1: now also J1.A5 (CC1); no longer J1.B5 (CC2)
- net at K1.2: now also D1.2 (A), Q1.3 (C); no longer D1.1 (K)
- net at R1.1: now also J1.B5 (CC2); no longer J1.A5 (CC1)
- net BOOT: now reaches SW2.2
- net BOOT: now also R3.1, U1.8 (IO9), C6.1; no longer R11.1
- removed net 3V3: R3.1, R4.1, R5.1, R6.1
- net D+: no longer names the net of J1.A6 (D+), J1.B6 (D+)
- net D+: now also U3.3 (I/O2); no longer U1.14 (IO19)
- net D-: no longer names the net of J1.A7 (D-), J1.B7 (D-)
- net D-: now also U3.1 (I/O1); no longer U1.13 (IO18)
- new net: J4.1 (Pin_1), Q2.1 (B), R13.1
- new net: R7.1, U4.1
- new net: D5.2 (A), R11.2
- new net: Q1.1 (B), R10.2
- new net: D2.2 (A), R14.1
- new net: C9.1, FB1.2, J1.A4 (VBUS), J1.A9 (VBUS), J1.B4 (VBUS), J1.B9 (VBUS), U3.5 (VBUS)
- new net: D4.2 (A), U4.2
- new net: U1.14 (IO19), U3.4 (I/O2)
- new net: U1.13 (IO18), U3.6 (I/O1)
- new net: R10.1, U4.3
- new net EN: C7.2, R5.1, SW1.2, U1.2 (EN)
Other:
- moved on the sheet: C1, C2, C3, D1, FB1, J1, J2, J3, J4, K1, R1, R10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

Commit message: new pcb design
Parts:
- C1, C2, C4, C6: footprint Capacitor_SMD:C_0805_2012Metric_Pad1.18x1.45mm_HandSolder -> Capacitor_SMD:C_0603_1608Metric_Pad1.08x0.95mm_HandSolder; LCSC C15850 -> C19702
- C10, C3, C5, C7: footprint Capacitor_SMD:C_0805_2012Metric_Pad1.18x1.45mm_HandSolder -> Capacitor_SMD:C_0603_1608Metric_Pad1.08x0.95mm_HandSolder; LCSC C28233 -> C14663
- C11: footprint (none) -> Capacitor_SMD:CP_Elec_4x5.4; LCSC (none) -> C970652
- C9: LCSC (none) -> C57112
- J2: footprint Connector_PinHeader_2.54mm:PinHeader_1x04_P2.54mm_Vertical -> Connector_PinSocket_2.54mm:PinSocket_1x04_P2.54mm_Vertical
- R1, R2: footprint Resistor_SMD:R_0805_2012Metric_Pad1.20x1.40mm_HandSolder -> Resistor_SMD:R_0603_1608Metric_Pad0.98x0.95mm_HandSolder; LCSC C27834 -> C23186
- R10: footprint Resistor_SMD:R_0805_2012Metric_Pad1.20x1.40mm_HandSolder -> Resistor_SMD:R_0603_1608Metric_Pad0.98x0.95mm_HandSolder; LCSC (none) -> C21190
- R11, R12, R14: footprint Resistor_SMD:R_0805_2012Metric_Pad1.20x1.40mm_HandSolder -> Resistor_SMD:R_0603_1608Metric_Pad0.98x0.95mm_HandSolder; LCSC C17557 -> C22962
- R13, R3, R4, R5, R6: footprint Resistor_SMD:R_0805_2012Metric_Pad1.20x1.40mm_HandSolder -> Resistor_SMD:R_0603_1608Metric_Pad0.98x0.95mm_HandSolder; LCSC C17414 -> C25804
- R7: footprint Resistor_SMD:R_0805_2012Metric_Pad1.20x1.40mm_HandSolder -> Resistor_SMD:R_0603_1608Metric_Pad0.98x0.95mm_HandSolder; LCSC (none) -> C22775
- R8, R9: value 2.1k -> 2.2k; footprint Resistor_SMD:R_0805_2012Metric_Pad1.20x1.40mm_HandSolder -> Resistor_SMD:R_0603_1608Metric_Pad0.98x0.95mm_HandSolder; LCSC C17517 -> C4190
- U3: LCSC (none) -> C2827654
- U4: LCSC (none) -> C5350
Changed lines of the file:
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@@
 			)
 		)
-		(property "Value" "2.1k"
+		(property "Value" "2.2k"
 			(at 240.03 91.44 0)
 			(effects
@@
 			)
 		)
-		(property "Footprint" "Resistor_SMD:R_0805_2012Metric_Pad1.20x1.40mm_HandSolder"
+		(property "Footprint" "Resistor_SMD:R_0603_1608Metric_Pad0.98x0.95mm_HandSolder"
 			(at 240.538 90.17 90)
 			(effects
@@
 			)
 		)
-		(property "LCSC" " C17517 "
+		(property "LCSC" "C4190"
 			(at 238.76 90.17 90)
 			(effects
@@
 			)
 		)
-		(property "Footprint" "Resistor_SMD:R_0805_2012Metric_Pad1.20x1.40mm_HandSolder"
+		(property "Footprint" "Resistor_SMD:R_0603_1608Metric_Pad0.98x0.95mm_HandSolder"
 			(at 193.04 120.142 90)
 			(effects
@@
 			)
 		)
-		(property "LCSC" ""
+		(property "LCSC" "C22775"
 			(at 193.04 121.92 90)
 			(effects
@@
 			)
 		)
-		(property "Footprint" "Capacitor_SMD:C_0805_2012Metric_Pad1.18x1.45mm_HandSolder"
+		(property "Footprint" "Capacitor_SMD:C_0603_1608Metric_Pad1.08x0.95mm_HandSolder"
 			(at 27.6352 34.29 0)
 			(effects
@@
 			)
 		)
-		(property "LCSC" "C15850"
+		(property "LCSC" "C19702"
 			(at 26.67 30.48 0)
 			(effects
@@
 			)
 		)
-		(property "Footprint" "Capacitor_SMD:C_0805_2012Metric_Pad1.18x1.45mm_HandSolder"
+		(property "Footprint" "Capacitor_SMD:C_0603_1608Metric_Pad1.08x0.95mm_HandSolder"
 			(at 153.67 37.1348 0)
 			(effects
@@
 			)
 		)
-		(property "LCSC" "C28233"
+		(property "LCSC" "C14663"
 			(at 149.86 38.1 0)
 			(effects
@@
 			)
 		)
-		(property "Footprint" "Resistor_SMD:R_0805_2012Metric_Pad1.20x1.40mm_HandSolder"
+		(property "Footprint" "Resistor_SMD:R_0603_1608Metric_Pad0.98x0.95mm_HandSolder"
 			(at 55.372 107.95 90)
 			(effects
@@
 			)
 		)
-		(property "LCSC" "C27834"
+		(property "LCSC" "C23186"
 			(at 57.15 107.95 90)
 			(effects
@@
 			)
 		)
-		(property "Footprint" "Capacitor_SMD:C_0805_2012Metric_Pad1.18x1.45mm_HandSolder"
+		(property "Footprint" "Capacitor_SMD:C_0603_1608Metric_Pad1.08x0.95mm_HandSolder"
 			(at 113.3348 125.73 0)
 			(effects
@@
 			)
 		)
-		(property "LCSC" "C28233"
+		(property "LCSC" "C14663"
 			(at 114.3 129.54 0)
 			(effects
@@
 			)
 		)
-		(property "Footprint" "Capacitor_SMD:C_0805_2012Metric_Pad1.18x1.45mm_HandSolder"
+		(property "Footprint" "Capacitor_SMD:C_0603_1608Metric_Pad1.08x0.95mm_HandSolder"
 			(at 65.7352 73.66 0)
 			(effects
@@
 			)
 		)
-		(property "LCSC" "C28233"
+		(property "LCSC" "C14663"
 			(at 64.77 69.85 0)
 			(effects
@@
 			)
 		)
-		(property "Footprint" "Capacitor_SMD:C_0805_2012Metric_Pad1.18x1.45mm_HandSolder"
+		(property "Footprint" "Capacitor_SMD:C_0603_1608Metric_Pad1.08x0.95mm_HandSolder"
 			(at 56.8452 34.29 0)
 			(effects
@@
 			)
 		)
-		(property "LCSC" "C15850"
+		(property "LCSC" "C19702"
 			(at 55.88 30.48 0)
 			(effects
@@
 			)
 		)
-		(property "Footprint" "Resistor_SMD:R_0805_2012Metric_Pad1.20x1.40mm_HandSolder"
+		(property "Footprint" "Resistor_SMD:R_0603_1608Metric_Pad0.98x0.95mm_HandSolder"
 			(at 116.078 119.38 90)
 			(effects
@@
 			)
 		)
-		(property "LCSC" " C17414 "
+		(property "LCSC" "C25804"
 			(at 114.3 119.38 90)
 			(effects
@@
 			)
 		)
+		(property "LCSC" "C57112"
+			(at 52.07 69.85 0)
+			(effects
+				(font
+					(size 1.27 1.27)
+				)
+				(hide yes)
+			)
+		)
 		(pin "2"
 		)
@@
 			)
 		)
-		(property "Footprint" "Resistor_SMD:R_0805_2012Metric_Pad1.20x1.40mm_HandSolder"
+		(property "Footprint" "Resistor_SMD:R_0603_1608Metric_Pad0.98x0.95mm_HandSolder"
 			(at 254 32.512 90)
 			(effects
@@
 			)
 		)
-		(property "LCSC" "C17557"
+		(property "LCSC" "C22962"
 			(at 254 34.29 90)
 			(effects
@@
 			)
 		)
-		(property "Footprint" "Resistor_SMD:R_0805_2012Metric_Pad1.20x1.40mm_HandSolder"
+		(property "Footprint" "Resistor_SMD:R_0603_1608Metric_Pad0.98x0.95mm_HandSolder"
 			(at 260.858 41.91 90)
 			(effects
@@
 			)
 		)
-		(property "LCSC" " C17414 "
+		(property "LCSC" "C25804"
 			(at 259.08 41.91 90)
 			(effects
@@
 			)
 		)
-		(property "Footprint" "Connector_PinHeader_2.54mm:PinHeader_1x04_P2.54mm_Vertical"
+		(property "Footprint" "Connector_PinSocket_2.54mm:PinSocket_1x04_P2.54mm_Vertical"
 			(at 266.7 91.44 0)
 			(effects
@@
 			)
 		)
-		(property "Value" "2.1k"
+		(property "Value" "2.2k"
 			(at 247.904 91.44 0)
 			(effects
@@
 			)
 		)
-		(property "Footprint" "Resistor_SMD:R_0805_2012Metric_Pad1.20x1.40mm_HandSolder"
+		(property "Footprint" "Resistor_SMD:R_0603_1608Metric_Pad0.98x0.95mm_HandSolder"
 			(at 248.158 90.17 90)
 			(effects
@@
 			)
 		)
-		(property "LCSC" " C17517 "
+		(property "LCSC" "C4190"
 			(at 246.38 90.17 90)
 			(effects
@@
 			)
 		)
+		(property "LCSC" "C2827654"
+			(at 64.77 96.52 0)
+			(effects
+				(font
+					(size 1.27 1.27)
+				)
+				(hide yes)
+			)
+		)
 		(pin "4"
 		)
@@
 			)
 		)
-		(property "Footprint" "Resistor_SMD:R_0805_2012Metric_Pad1.20x1.40mm_HandSolder"
+		(property "Footprint" "Resistor_SMD:R_0603_1608Metric_Pad0.98x0.95mm_HandSolder"
 			(at 89.408 30.48 90)
 			(effects
@@
 			)
 		)
-		(property "LCSC" "C17557"
+		(property "LCSC" "C22962"
 			(at 87.63 30.48 90)
 			(effects
@@
 			)
 		)
-		(property "Footprint" "Resistor_SMD:R_0805_2012Metric_Pad1.20x1.40mm_HandSolder"
+		(property "Footprint" "Resistor_SMD:R_0603_1608Metric_Pad0.98x0.95mm_HandSolder"
 			(at 90.678 119.38 90)
 			(effects
@@
 			)
 		)
-		(property "LCSC" " C17414 "
+		(property "LCSC" "C25804"
 			(at 88.9 119.38 90)
 			(effects
@@
 			)
 		)
-		(property "Footprint" "Resistor_SMD:R_0805_2012Metric_Pad1.20x1.40mm_HandSolder"
+		(property "Footprint" "Resistor_SMD:R_0603_1608Metric_Pad0.98x0.95mm_HandSolder"
 			(at 116.84 75.438 90)
 			(effects
@@
 			)
 		)
-		(property "LCSC" " C17414 "
+		(property "LCSC" "C25804"
 			(at 116.84 73.66 90)
 			(effects
@@
 			)
 		)
-		(property "Footprint" "Capacitor_SMD:C_0805_2012Metric_Pad1.18x1.45mm_HandSolder"
+		(property "Footprint" "Capacitor_SMD:C_0603_1608Metric_Pad1.08x0.95mm_HandSolder"
 			(at 89.8652 133.35 0)
 			(effects
@@
 			)
 		)
-		(property "LCSC" "C15850"
+		(property "LCSC" "C19702"
 			(at 88.9 129.54 0)
 			(effects
@@
 			)
 		)
-		(property "Footprint" "Resistor_SMD:R_0805_2012Metric_Pad1.20x1.40mm_HandSolder"
+		(property "Footprint" "Resistor_SMD:R_0603_1608Metric_Pad0.98x0.95mm_HandSolder"
 			(at 46.482 107.95 90)
 			(effects
@@
 			)
 		)
-		(property "LCSC" "C27834"
+		(property "LCSC" "C23186"
 			(at 48.26 107.95 90)
 			(effects
@@
 			)
 		)
-		(property "Footprint" "Capacitor_SMD:C_0805_2012Metric_Pad1.18x1.45mm_HandSolder"
+		(property "Footprint" "Capacitor_SMD:C_0603_1608Metric_Pad1.08x0.95mm_HandSolder"
 			(at 68.2752 34.29 0)
 			(effects
@@
 			)
 		)
-		(property "LCSC" "C28233"
+		(property "LCSC" "C14663"
 			(at 67.31 30.48 0)
 			(effects
@@
 			)
 		)
-		(property "Footprint" "Resistor_SMD:R_0805_2012Metric_Pad1.20x1.40mm_HandSolder"
+		(property "Footprint" "Resistor_SMD:R_0603_1608Metric_Pad0.98x0.95mm_HandSolder"
 			(at 221.488 130.81 90)
 			(effects
@@
 			)
 		)
-		(property "LCSC" ""
+		(property "LCSC" "C21190"
 			(at 219.71 130.81 90)
 			(effects
@@
 			)
 		)
-		(property "Footprint" "Capacitor_SMD:C_0805_2012Metric_Pad1.18x1.45mm_HandSolder"
+		(property "Footprint" "Capacitor_SMD:C_0603_1608Metric_Pad1.08x0.95mm_HandSolder"
 			(at 153.67 49.8348 0)
 			(effects
@@
 			)
 		)
-		(property "LCSC" "C15850"
+		(property "LCSC" "C19702"
 			(at 149.86 50.8 0)
 			(effects
@@
 			)
 		)
-		(property "Footprint" ""
+		(property "Footprint" "Capacitor_SMD:CP_Elec_4x5.4"
 			(at 79.7052 73.66 0)
 			(effects
@@
 			)
 		)
+		(property "LCSC" "C970652"
+			(at 78.74 69.85 0)
+			(effects
+				(font
+					(size 1.27 1.27)
+				)
+				(hide yes)
+			)
+		)
 		(pin "1"
 		)
@@
 			)
 		)
-		(property "Footprint" "Resistor_SMD:R_0805_2012Metric_Pad1.20x1.40mm_HandSolder"
+		(property "Footprint" "Resistor_SMD:R_0603_1608Metric_Pad0.98x0.95mm_HandSolder"
 			(at 116.84 90.678 90)
 			(effects
@@
 			)
 		)
-		(property "LCSC" " C17414 "
+		(property "LCSC" "C25804"
 			(at 116.84 88.9 90)
 			(effects
@@
 			)
 		)
+		(property "LCSC" "C5350"
+			(at 207.01 124.46 0)
+			(effects
+				(font
+					(size 1.27 1.27)
+				)
+				(hide yes)
+			)
+		)
 		(pin "4"
 		)
@@
 			)
 		)
-		(property "Footprint" "Resistor_SMD:R_0805_2012Metric_Pad1.20x1.40mm_HandSolder"
+		(property "Footprint" "Resistor_SMD:R_0603_1608Metric_Pad0.98x0.95mm_HandSolder"
 			(at 104.648 30.48 90)
 			(effects
@@
 			)
 		)
-		(property "LCSC" "C17557"
+		(property "LCSC" "C22962"
 			(at 102.87 30.48 90)
 			(effects

Commit message: I like this but want to invert my input LEDs
Parts:
- removed C3: 100nF, Capacitor_SMD:C_0603_1608Metric_Pad1.08x0.95mm_HandSolder, symbol Device:C
- removed J1: USB_C_Receptacle_USB2.0_14P, Connector_USB:USB_C_Receptacle_HCTL_HC-TYPE-C-16P-01A, symbol Connector:USB_C_Receptacle_USB2.0_14P
- removed J2: AHT21, Connector_PinSocket_2.54mm:PinSocket_1x04_P2.54mm_Vertical, symbol Connector:Conn_01x04_Socket
- removed R1, R2: 5.1k, Resistor_SMD:R_0603_1608Metric_Pad0.98x0.95mm_HandSolder, symbol Device:R
- removed R10: 1k, Resistor_SMD:R_0603_1608Metric_Pad0.98x0.95mm_HandSolder, symbol Device:R
- added C8: 100nF, Capacitor_SMD:C_0402_1005Metric_Pad0.74x0.62mm_HandSolder, symbol Device:C
- added D3: GREEN LED, LED_SMD:LED_0603_1608Metric_Pad1.05x0.95mm_HandSolder, symbol Device:LED
- added J1: USB_B_Mini, Connector_USB:USB_Mini-B_Lumberg_2486_01_Horizontal, symbol Connector:USB_B_Mini
- added J2: ~, Connector_Molex:Molex_Micro-Fit_3.0_43650-0200_1x02_P3.00mm_Horizontal, symbol Connector:Conn_01x02_Socket
- added Q1: SS8050, Package_TO_SOT_SMD:SOT-23, symbol Transistor_BJT:SS8050
- added R11, R14: 10k, Resistor_SMD:R_0603_1608Metric_Pad0.98x0.95mm_HandSolder, symbol Device:R
- added R15: 1k, Resistor_SMD:R_0603_1608Metric_Pad0.98x0.95mm_HandSolder, symbol Device:R
- added R9: 220, Resistor_SMD:R_0603_1608Metric_Pad0.98x0.95mm_HandSolder, symbol Device:R
- added U3: SHT4x, Sensor_Humidity:Sensirion_DFN-4_1.5x1.5mm_P0.8mm_SHT4x_NoCentralPad, symbol Sensor_Humidity:SHT4x
- C2: value 10uF -> 22uF; LCSC C19702 -> C59461
- J3: renamed from J4; value DOOR SW -> ~; LCSC C192562 -> C122431
- J4: renamed from J3; value DOOR CTL -> ~; LCSC C192562 -> C122431
- renumbered C7 to C10, C5 to C3, C9 to C5, C10 to C6, C11 to C7, C6 to C9, D2 to D1, D3 to D2, D5 to D4, D1 to D5, D4 to D6, Q1 to Q3, R14 to R1, R11 to R10, R13 to R12, R7 to R13, R12 to R2, R4 to R3, R3 to R4, R8 to R6, R9 to R7, R6 to R8, SW2 to SW1, SW1 to SW2, U2 to U1, U1 to U2, U3 to U4, U4 to U5
Connections:
- net +3V3: now also C8.2, R11.2, R9.1, U3.3 (VDD)
- net BOOT: now also C10.2, R5.1, SW2.2; no longer C9.1, R4.1, SW1.2
- net EN: now also C9.1, R4.1, SW1.2; no longer C10.2, R5.1, SW2.2
- net GND: now also J3.1 (Pin_1), C8.1, J1.5 (GND), J2.1 (Pin_1), Q1.2 (E), R14.1, U3.4 (VSS); no longer J3.2 (Pin_2)
- net RELAY: now also U2.10 (IO10), R14.2; no longer U2.6 (IO7)
- net SCL: now also U3.2 (SCL)
- net SDA: now also U3.1 (SDA)
- net at Q2.1 (B), R12.1: now also J3.2 (Pin_2); no longer J3.1 (Pin_1)
- net at Q3.1 (B): now also R15.1
- net at C5.1, FB1.2, U4.5 (VBUS): now also J1.1 (VBUS)
- net at U5.3: now also R15.2
- net SW renamed IN2
- net IN2: now also U2.6 (IO7); no longer U2.5 (IO6)
- new net: J2.2 (Pin_2), Q1.1 (B), R11.1
- new net: D3.2 (A), R9.2
- new net IN1: D3.1 (K), Q1.3 (C), U2.5 (IO6)
Other:
- moved on the sheet: C1, C10, C2, C5, C6, C7, C9, D1, D2, D4, D5, D6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
